File: deltas_backplane.kicad_pcb (KiCad board)
At the start: 2 copper layers, 140.6 x 119.4 mm, 11 parts, among them J1 SNP_female_straight, J2 SNP_female_straight, J3 SNP_female_straight, J4 SNP_female_straight, J5 SNP_male_angle, J6 zx_bus, J7 zx_bus, J8 Barrel_Jack, SW1 SW_SPDT

Commit message: 03.10.2023 update
Parts:
- removed SW1: SW_SPDT, Backplane:MTS-102-C3
- added J9: Conn_01x04, Backplane_2:PinHeader_1x04_P2.54mm_Vertical, F.Cu at (118.0, 29.2)
- added JP1: Jumper_3_Open, Backplane_2:PinHeader_1x03_P2.54mm_Vertical, F.Cu at (133.5, 31.8)
- C1: footprint Capacitor_THT:CP_Radial_Tantal_D7.0mm_P5.00mm -> Backplane_2:CP_Radial_D8.0mm_P5.00mm
- C2: footprint Capacitor_THT:C_Disc_D5.0mm_W2.5mm_P5.00mm -> Backplane_2:C_Disc_D5.0mm_W2.5mm_P5.00mm
- J1: footprint Backplane:snp_straight -> Backplane_2:snp_straight
- J2, J3, J4: footprint Backplane:snp59_96_male_straight -> Backplane_2:snp59_96_male_straight
- J5: footprint Backplane:snp59_96_female_angle_3 -> Backplane_2:snp59_96_female_angle_3
- J6: footprint Backplane:ZX SPECTRUM EDGE CONNECTOR (HORIZONTAL) -> Backplane_2:ZX SPECTRUM EDGE CONNECTOR (HORIZONTAL)
- J7: footprint Backplane:Spectrum_edge_slot_FIXED -> Backplane_2:Spectrum_edge_slot_FIXED
- J8: footprint Backplane:BarrelJack_GCT_DCJ200-10-A_Horizontal -> Backplane_2:BarrelJack_GCT_DCJ200-10-A_Horizontal
- moved J2 52.5 mm to (128.3, 46.2)
- moved J3 52.5 mm to (155.0, 46.2)
- moved J7 52.5 mm to (200.9, 84.2)
- moved J1 52.5 mm to (98.5, 124.3)
- moved J4 52.5 mm to (181.7, 46.2)
- moved J5 52.5 mm to (222.7, 46.0)
- moved J8 41.7 mm to (136.6, 25.4), turned to 180 degrees
- moved C1 39.3 mm to (127.9, 26.6), turned to 180 degrees
- moved J6 39.2 mm to (190.8, 20.7)
- moved C2 37.6 mm to (127.9, 20.1), turned to 180 degrees
Routing:
- net A6: track 279.9 -> 212.9 mm, vias 2 -> 3
- net ЧТПЗУL: track 171.6 -> 222.4 mm
- net B21_SNP: track 131.2 -> 180.0 mm, vias 0 -> 1
- net ЗПL: track 211.1 -> 256.4 mm, vias 1 -> 3
- net GND: track 436.5 -> 479.3 mm
- net D5: track 176.5 -> 213.2 mm, vias 2 -> 3
- net СТОПL: track 263.7 -> 227.1 mm, vias 5 -> 1
- net НПРL: track 260.4 -> 225.2 mm, vias 5 -> 1
- net ОЗУL: track 197.1 -> 230.6 mm, vias 2 -> 0
- net ОЖИДL: track 240.3 -> 207.6 mm, vias 4 -> 1
- net ПРL: track 188.1 -> 218.6 mm, vias 1 -> 0
- net D2: track 207.6 -> 177.9 mm
- net A12: track 193.0 -> 163.6 mm, vias 2 -> 1
- net A3: track 217.3 -> 188.6 mm
- net D3: track 212.3 -> 185.0 mm, vias 4 -> 1
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Other:
- board size 140.6 x 119.4 mm -> 143.5 x 119.2 mm

Commit message: Update 09.10.2023
Parts:
- added H1: MountingHole_2.5mm, MountingHole:MountingHole_2.5mm, F.Cu at (166.6, 30.5)
- added H2: MountingHole_2.5mm, MountingHole:MountingHole_2.5mm, F.Cu at (166.6, 130.0)
- added H3: MountingHole_2.5mm, MountingHole:MountingHole_2.5mm, F.Cu at (212.3, 30.5)
- added H4: MountingHole_2.5mm, MountingHole:MountingHole_2.5mm, F.Cu at (212.3, 130.0)
- J8: value Barrel_Jack -> Ext. Power (5V)
Routing:
- net GND: track 479.3 -> 483.3 mm, vias 3 -> 46
- net M1L: track 224.9 -> 223.5 mm
- net A10: track 226.8 -> 226.0 mm
- net РГНL: track 224.3 -> 223.6 mm
- net A3: track 188.6 -> 187.8 mm
- net A1: track 184.1 -> 183.4 mm
- net A2: track 186.7 -> 186.0 mm
- net A0: track 180.4 -> 179.7 mm
- added copper zone on B.Cu, net GND
- added copper zone on F.Cu, net GND

Commit message: Update deltas_backplane.kicad_pcb
Other:
- board size 143.5 x 119.2 mm -> 143.5 x 118.8 mm
Changed lines of the file:
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@@
   (gr_line (start 167.74399 25.64352) (end 165.71199 25.64352)
     (stroke (width 0.1) (type solid)) (layer "Edge.Cuts"))
-  (gr_line (start 228.70399 135.47501) (end 85.19798 135.47501)
+  (gr_line (start 228.70399 135) (end 85.19798 135)
     (stroke (width 0.1) (type default)) (layer "Edge.Cuts"))
   (gr_arc (start 153.01199 17.24552) (mid 153.30488 16.538407) (end 154.01199 16.24552)
@@
   (gr_line (start 167.74399 16.24552) (end 167.74399 25.64352)
     (stroke (width 0.1) (type solid)) (layer "Edge.Cuts"))
-  (gr_line (start 227.70399 16.24552) (end 167.74399 16.24552)
+  (gr_line (start 228.70399 16.24552) (end 167.74399 16.24552)
     (stroke (width 0.1) (type solid)) (layer "Edge.Cuts"))
   (gr_line (start 115 36.30402) (end 115 16.56352)
     (stroke (width 0.1) (type default)) (layer "Edge.Cuts"))
-  (gr_line (start 228.70399 30.17701) (end 228.70399 135.47501)
+  (gr_line (start 228.70399 16.24552) (end 228.70399 135)
     (stroke (width 0.1) (type default)) (layer "Edge.Cuts"))
-  (gr_line (start 85.19798 36.30402) (end 85.19798 135.47501)
-    (stroke (width 0.1) (type solid)) (layer "Edge.Cuts"))
-  (gr_line (start 228.70399 30.17701) (end 228.70399 17.24552)
+  (gr_line (start 85.19798 36.30402) (end 85.19798 135)
     (stroke (width 0.1) (type solid)) (layer "Edge.Cuts"))
   (gr_line (start 85.19798 36.30402) (end 115 36.30402)
     (stroke (width 0.1) (type default)) (layer "Edge.Cuts"))
-  (gr_arc (start 227.70399 16.24552) (mid 228.411093 16.538414) (end 228.70399 17.24552)
-    (stroke (width 0.1) (type default)) (layer "Edge.Cuts"))
   (gr_line (start 142.39299 16.56352) (end 142.39299 30.17701)

Commit message: Gerbers upload
Parts:
- C1: value 1000uF 10V -> 1000uF 16V
Other:
- board text added: "+5"
- board text added: "1"
- board text added: "3"
- board text added: "Delta Pwr."
- board text added: "Ext.Pwr"
- board text added: "GND"
- board text added: "JP1 jumper: 1-2 - internal +5V power 2-3 - external power"
- board text added: "{dblquote}Дельта-С{dblquote} - бекплейн Version 0.1 Board Design by MadCat, 2023 https://github.com/madcatse/Delta-S-backplane t.me/zx_delta_s"

Commit message: Small update (0.1.1)
Routing:
- net GND: track 483.3 -> 258.4 mm, vias 46 -> 24
- net B19_SNP: track 198.5 -> 135.0 mm
- net ЗПL: track 256.4 -> 206.2 mm, vias 3 -> 2
- net B21_SNP: track 180.0 -> 139.0 mm, vias 1 -> 4
- net НПРL: track 225.2 -> 192.9 mm
- net СТОПL: track 227.1 -> 195.2 mm
- net ПРL: track 218.6 -> 188.0 mm, vias 0 -> 1
- net B28_SNP: track 131.5 -> 161.8 mm, vias 0 -> 3
- net ОЗУL: track 230.6 -> 201.3 mm, vias 0 -> 1
- net D5: track 213.2 -> 188.2 mm, vias 3 -> 1
- net A0: track 179.7 -> 199.8 mm, vias 2 -> 1
- net D6: track 183.4 -> 202.8 mm, vias 2 -> 4
- net A8: track 227.3 -> 246.1 mm, vias 2 -> 3
- net A1: track 183.4 -> 197.7 mm, vias 2 -> 3
- net A19_SNP: track 133.7 -> 145.5 mm, vias 0 -> 3
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Other:
- board size 143.5 x 118.8 mm -> 143 x 118.8 mm

Commit message: Version 0.2 upload
Parts:
- removed H1, H2, H3, H4: MountingHole_2.5mm, MountingHole:MountingHole_2.5mm
- added M31: MountingHole_3.2mm_M3, MountingHole:MountingHole_3.2mm_M3, F.Cu at (211.5, 129.3)
- added M31: MountingHole_3.2mm_M3, MountingHole:MountingHole_3.2mm_M3, F.Cu at (165.5, 129.3)
- added M31: MountingHole_3.2mm_M3, MountingHole:MountingHole_3.2mm_M3, F.Cu at (211.5, 32.8)
- added M31: MountingHole_3.2mm_M3, MountingHole:MountingHole_3.2mm_M3, F.Cu at (165.5, 32.8)
- C1: value 1000uF 16V -> 1000uF 10V
- J1: value SNP_female_straight -> СНП59-64 94х118 20-2-Р
- J2, J3, J4: value SNP_female_straight -> СНП59-64 94х118-21-2-В
- J5: value SNP_male_angle -> СНП59-64 94х118 23-2-В
- J6: value zx_bus -> ZX-BUS
- J7: value zx_bus -> EDGE Connector SL56
- J8: value Ext. Power (5V) -> Barrel_Jack
- moved J7 2.98 mm to (198.0, 84.4)
Connections:
- J6 pad 28: B32_SNP -> unconnected-(J6-NC-Pad28)
- J7 pad 28: B32_SNP -> unconnected-(J7-NC-Pad28)
- J7 pad 41: unconnected-(J7-NC-Pad41) -> B28_SNP
Routing:
- net GND: track 258.4 -> 3.05 mm, vias 24 -> 47
- net B32_SNP: track 254.8 -> 129.9 mm, vias 1 -> 0
- net A19_SNP: track 145.5 -> 211.5 mm, vias 3 -> 1
- net 5V_connector: track 207.4 -> 238.9 mm, vias 2 -> 3
- net B28_SNP: track 161.8 -> 180.8 mm, vias 3 -> 2
- net D6: track 202.8 -> 221.2 mm, vias 4 -> 2
- net A0: track 199.8 -> 182.2 mm
- net ВУL: track 202.6 -> 218.9 mm, vias 1 -> 7
- net ЗПL: track 206.2 -> 221.4 mm, vias 2 -> 3
- net ПЗШL: track 223.4 -> 238.2 mm, vias 0 -> 4
- net A7: track 225.6 -> 211.3 mm, vias 2 -> 1
- net A1: track 197.7 -> 184.1 mm
- net D3: track 193.4 -> 182.4 mm
- net A10: track 227.7 -> 236.5 mm, vias 2 -> 3
- net A5: track 227.9 -> 219.1 mm, vias 4 -> 1
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Other:
- outline, holes or cut-outs redrawn
- board text added: "A"
- board text added: "B"
- board text added: "C"
- board text added: "{dblquote}Дельта-С{dblquote} - бекплейн Version 0.2 Board Design by MadCat, 2026 https://github.com/madcatse/Delta-S-backplane t.me/zx_delta_s"
- board text removed: "{dblquote}Дельта-С{dblquote} - бекплейн Version 0.1 Board Design by MadCat, 2023 https://github.com/madcatse/Delta-S-backplane t.me/zx_delta_s"
