File: deltas_backplane.kicad_sch (KiCad schematic)
At the start: 11 parts, among them J1 SNP_female_straight, J2 SNP_female_straight, J3 SNP_female_straight, J4 SNP_female_straight, J5 SNP_male_angle, J6 zx_bus, J7 zx_bus, J8 Barrel_Jack, SW1 SW_SPDT

Commit message: Power fix
Parts:
- J8: footprint Connector_BarrelJack:BarrelJack_SwitchcraftConxall_RAPC10U_Horizontal -> Backplane:BarrelJack_GCT_DCJ200-10-A_Horizontal
- SW1: footprint Button_Switch_SMD:SW_DPDT_CK_JS202011JCQN -> Backplane:MTS-102-C3
Changed lines of the file:
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@@
 (kicad_sch (version 20230121) (generator eeschema)
   (paper "A4")
+  (junction (at 255.27 137.16) (diameter 0) (color 0 0 0 0)
+  )
   (junction (at 222.25 134.62) (diameter 0) (color 0 0 0 0)
   )
   (junction (at 209.55 134.62) (diameter 0) (color 0 0 0 0)
   )
+  (junction (at 215.9 134.62) (diameter 0) (color 0 0 0 0)
+  )
+  (junction (at 241.3 139.7) (diameter 0) (color 0 0 0 0)
+  )
   (junction (at 146.05 134.62) (diameter 0) (color 0 0 0 0)
   )
@@
     (stroke (width 0) (type default))
   )
-  (wire (pts (xy 209.55 134.62) (xy 222.25 134.62))
+  (wire (pts (xy 209.55 134.62) (xy 215.9 134.62))
     (stroke (width 0) (type default))
   )
@@
     (stroke (width 0) (type default))
   )
+  (wire (pts (xy 215.9 134.62) (xy 222.25 134.62))
+    (stroke (width 0) (type default))
+  )
   (wire (pts (xy 81.28 96.52) (xy 86.36 96.52))
     (stroke (width 0) (type default))
@@
     (stroke (width 0) (type default))
   )
-  (wire (pts (xy 238.76 139.7) (xy 242.57 139.7))
+  (wire (pts (xy 238.76 139.7) (xy 241.3 139.7))
     (stroke (width 0) (type default))
   )
@@
     (stroke (width 0) (type default))
   )
-  (wire (pts (xy 257.81 137.16) (xy 252.73 137.16))
+  (wire (pts (xy 257.81 137.16) (xy 255.27 137.16))
     (stroke (width 0) (type default))
   )
@@
     (stroke (width 0) (type default))
   )
+  (wire (pts (xy 241.3 139.7) (xy 242.57 139.7))
+    (stroke (width 0) (type default))
+  )
   (wire (pts (xy 55.88 81.28) (xy 50.8 81.28))
     (stroke (width 0) (type default))
@@
     (stroke (width 0) (type default))
   )
+  (wire (pts (xy 255.27 137.16) (xy 252.73 137.16))
+    (stroke (width 0) (type default))
+  )
   (wire (pts (xy 240.03 106.68) (xy 246.38 106.68))
     (stroke (width 0) (type default))
@@
     )
   )
+  (netclass_flag "" (length 2.54) (shape round) (at 227.33 134.62 0) (fields_autoplaced)
+    (effects (font (size 1.27 1.27)) (justify left bottom))
+    (property "Netclass" "power" (at 228.0285 132.08 0)
+      (effects (font (size 1.27 1.27) italic) (justify left))
+    )
+  )
   (symbol (lib_id "power:GND") (at 55.88 43.18 90) (mirror x) (unit 1)
     (in_bom yes) (on_board yes) (dnp no)
@@
       (effects (font (size 1.27 1.27)))
     )
-    (property "Footprint" "Connector_BarrelJack:BarrelJack_SwitchcraftConxall_RAPC10U_Horizontal" (at 195.58 138.176 0)
+    (property "Footprint" "Backplane:BarrelJack_GCT_DCJ200-10-A_Horizontal" (at 195.58 138.176 0)
       (effects (font (size 1.27 1.27)) hide)
     )
@@
       (effects (font (size 1.27 1.27)))
     )
-    (property "Footprint" "Button_Switch_SMD:SW_DPDT_CK_JS202011JCQN" (at 247.65 137.16 0)
+    (property "Footprint" "Backplane:MTS-102-C3" (at 247.65 137.16 0)
       (effects (font (size 1.27 1.27)) hide)
     )
@@
     )
   )
+  (symbol (lib_id "power:PWR_FLAG") (at 255.27 137.16 0) (unit 1)
+    (in_bom yes) (on_board yes) (dnp no) (fields_autoplaced)
+    (property "Reference" "#FLG03" (at 255.27 135.255 0)
+      (effects (font (size 1.27 1.27)) hide)
+    )
+    (property "Value" "PWR_FLAG" (at 255.27 133.35 0)
+      (effects (font (size 1.27 1.27)))
+    )
+    (property "Footprint" "" (at 255.27 137.16 0)
+      (effects (font (size 1.27 1.27)) hide)
+    )
+    (property "Datasheet" "~" (at 255.27 137.16 0)
+      (effects (font (size 1.27 1.27)) hide)
+    )
+    (pin "1")
+    (instances
+      (project "deltas_backplane"
+        (path "/a9508c3f-c02b-458d-89a9-c2b48f8b1580"
+          (reference "#FLG03") (unit 1)
+        )
+      )
+    )
+  )
   (symbol (lib_id "power:GND") (at 222.25 142.24 0) (mirror y) (unit 1)
     (in_bom yes) (on_board yes) (dnp no)
@@
     )
   )
+  (symbol (lib_id "power:PWR_FLAG") (at 241.3 139.7 0) (unit 1)
+    (in_bom yes) (on_board yes) (dnp no) (fields_autoplaced)
+    (property "Reference" "#FLG04" (at 241.3 137.795 0)
+      (effects (font (size 1.27 1.27)) hide)
+    )
+    (property "Value" "PWR_FLAG" (at 241.3 135.89 0)
+      (effects (font (size 1.27 1.27)))
+    )
+    (property "Footprint" "" (at 241.3 139.7 0)
+      (effects (font (size 1.27 1.27)) hide)
+    )
+    (property "Datasheet" "~" (at 241.3 139.7 0)
+      (effects (font (size 1.27 1.27)) hide)
+    )
+    (pin "1")
+    (instances
+      (project "deltas_backplane"
+        (path "/a9508c3f-c02b-458d-89a9-c2b48f8b1580"
+          (reference "#FLG04") (unit 1)
+        )
+      )
+    )
+  )
   (symbol (lib_id "power:GND") (at 109.22 40.64 90) (mirror x) (unit 1)
     (in_bom yes) (on_board yes) (dnp no)
@@
         )
       )
+    )
+  )
+  (symbol (lib_id "power:PWR_FLAG") (at 215.9 134.62 0) (unit 1)
+    (in_bom yes) (on_board yes) (dnp no) (fields_autoplaced)
+    (property "Reference" "#FLG02" (at 215.9 132.715 0)
+      (effects (font (size 1.27 1.27)) hide)
+    )
+    (property "Value" "PWR_FLAG" (at 215.9 130.81 0)
+      (effects (font (size 1.27 1.27)))
+    )
+    (property "Footprint" "" (at 215.9 134.62 0)
+      (effects (font (size 1.27 1.27)) hide)
+    )
+    (property "Datasheet" "~" (at 215.9 134.62 0)
+      (effects (font (size 1.27 1.27)) hide)
+    )
+    (pin "1")
+    (instances
+      (project "deltas_backplane"
+        (path "/a9508c3f-c02b-458d-89a9-c2b48f8b1580"
+          (reference "#FLG02") (unit 1)
+        )
+      )

Commit message: 03.10.2023 update
Parts:
- removed SW1: SW_SPDT, Backplane:MTS-102-C3, symbol Switch:SW_SPDT
- added J9: Conn_01x04, Connector_PinHeader_2.54mm:PinHeader_1x04_P2.54mm_Vertical, symbol Connector_Generic:Conn_01x04
- added JP1: Jumper_3_Open, Connector_PinHeader_2.54mm:PinHeader_1x03_P2.54mm_Vertical, symbol Jumper:Jumper_3_Open
- C1: footprint Capacitor_THT:CP_Radial_Tantal_D7.0mm_P5.00mm -> Capacitor_THT:CP_Radial_D8.0mm_P5.00mm; symbol Device:C_Polarized -> backplane_2:C_Polarized
- C2: symbol Device:C -> backplane_2:C
- J1, J2, J3, J4: symbol backplane:SNP_female_straight -> backplane_2:SNP_female_straight
- J5: symbol backplane:SNP_male_angle -> backplane_2:SNP_male_angle
- J6, J7: symbol backplane:zx_bus -> backplane_2:zx_bus
- J8: symbol Connector:Barrel_Jack -> backplane_2:Barrel_Jack
Connections:
- net +5V: now also JP1.1 (A)
- net 5V_connector: now also J9.1 (Pin_1), JP1.2 (C)
- net GND: now also J9.2 (Pin_2)
- net at C1.1, C2.1, J8.1: now also JP1.3 (B)
- no-connect marks 12 -> 14

Commit message: Version 0.2 upload
Parts:
- C1: footprint Capacitor_THT:CP_Radial_D8.0mm_P5.00mm -> Backplane_2:CP_Radial_D8.0mm_P5.00mm
- C2: footprint Capacitor_THT:C_Disc_D5.0mm_W2.5mm_P5.00mm -> Backplane_2:C_Disc_D5.0mm_W2.5mm_P5.00mm
- J1: footprint Backplane:snp_straight -> Backplane_2:snp_straight
- J2, J3, J4: footprint Backplane:snp59_96_male_straight -> Backplane_2:snp59_96_male_straight
- J5: footprint Backplane:snp59_96_female_angle_3 -> Backplane_2:snp59_96_female_angle_3
- J6: footprint Backplane:ZX SPECTRUM EDGE CONNECTOR (HORIZONTAL) -> Backplane_2:ZX SPECTRUM EDGE CONNECTOR (HORIZONTAL)
- J7: footprint Backplane:Spectrum_edge_slot_FIXED -> Backplane_2:Spectrum_edge_slot_FIXED
- J8: footprint Backplane:BarrelJack_GCT_DCJ200-10-A_Horizontal -> Backplane_2:BarrelJack_GCT_DCJ200-10-A_Horizontal
- J9: footprint Connector_PinHeader_2.54mm:PinHeader_1x04_P2.54mm_Vertical -> Backplane_2:PinHeader_1x04_P2.54mm_Vertical
- JP1: footprint Connector_PinHeader_2.54mm:PinHeader_1x03_P2.54mm_Vertical -> Backplane_2:PinHeader_1x03_P2.54mm_Vertical
Connections:
- net B28_SNP: now also J7.41 (NC)
- net B32_SNP: no longer J6.28 (NC), J7.28 (NC)
- no-connect marks 14 -> 16
Changed lines of the file:
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@@
   (no_connect (at 57.15 175.26))
   (no_connect (at 118.11 175.26))
+  (no_connect (at 57.15 190.5))
   (no_connect (at 57.15 177.8))
   (no_connect (at 253.365 155.575))
+  (no_connect (at 118.11 190.5))
   (no_connect (at 140.97 157.48))
   (no_connect (at 80.01 157.48))
@@
     (stroke (width 0) (type default))
   )
-  (wire (pts (xy 50.8 190.5) (xy 57.15 190.5))
-    (stroke (width 0) (type default))
-  )
   (wire (pts (xy 209.55 109.22) (xy 214.63 109.22))
     (stroke (width 0) (type default))
@@
     (stroke (width 0) (type default))
   )
+  (wire (pts (xy 140.97 152.4) (xy 147.955 152.4))
+    (stroke (width 0) (type default))
+  )
   (wire (pts (xy 240.03 58.42) (xy 246.38 58.42))
     (stroke (width 0) (type default))
@@
     (stroke (width 0) (type default))
   )
-  (wire (pts (xy 111.76 190.5) (xy 118.11 190.5))
-    (stroke (width 0) (type default))
-  )
   (wire (pts (xy 146.05 134.62) (xy 140.97 134.62))
     (stroke (width 0) (type default))
@@
     )
   )
-  (global_label "B32_SNP" (shape input) (at 50.8 190.5 180) (fields_autoplaced)
-    (effects (font (size 1.27 1.27)) (justify right))
-    (property "Intersheetrefs" "${INTERSHEET_REFS}" (at 39.9202 190.4206 0)
-      (effects (font (size 1.27 1.27)) (justify right) hide)
-    )
-  )
   (global_label "A28_SNP" (shape input) (at 214.63 99.06 0) (fields_autoplaced)
     (effects (font (size 1.27 1.27)) (justify left))
@@
     )
   )
+  (global_label "B28_SNP" (shape input) (at 147.955 152.4 0) (fields_autoplaced)
+    (effects (font (size 1.27 1.27)) (justify left))
+    (property "Intersheetrefs" "${INTERSHEET_REFS}" (at 159.4068 152.4 0)
+      (effects (font (size 1.27 1.27)) (justify left) hide)
+    )
+  )
   (global_label "A8" (shape input) (at 132.08 91.44 180) (fields_autoplaced)
     (effects (font (size 1.27 1.27)) (justify right))
@@
     )
   )
-  (global_label "B32_SNP" (shape input) (at 111.76 190.5 180) (fields_autoplaced)
-    (effects (font (size 1.27 1.27)) (justify right))
-    (property "Intersheetrefs" "${INTERSHEET_REFS}" (at 100.8802 190.4206 0)
-      (effects (font (size 1.27 1.27)) (justify right) hide)
-    )
-  )
   (global_label "ПЗШL" (shape input) (at 161.29 91.44 0) (fields_autoplaced)
     (effects (font (size 1.27 1.27)) (justify left))
@@
       (effects (font (size 1.27 1.27)))
     )
-    (property "Footprint" "Backplane:BarrelJack_GCT_DCJ200-10-A_Horizontal" (at 195.58 138.176 0)
+    (property "Footprint" "Backplane_2:BarrelJack_GCT_DCJ200-10-A_Horizontal" (at 195.58 138.176 0)
       (effects (font (size 1.27 1.27)) hide)
     )
@@
       (effects (font (size 1.27 1.27)) (justify left))
     )
-    (property "Footprint" "Capacitor_THT:C_Disc_D5.0mm_W2.5mm_P5.00mm" (at 223.2152 142.24 0)
+    (property "Footprint" "Backplane_2:C_Disc_D5.0mm_W2.5mm_P5.00mm" (at 223.2152 142.24 0)
       (effects (font (size 1.27 1.27)) hide)
     )
@@
       (effects (font (size 1.27 1.27)))
     )
-    (property "Footprint" "Backplane:snp59_96_male_straight" (at 200.66 24.13 0)
+    (property "Footprint" "Backplane_2:snp59_96_male_straight" (at 200.66 24.13 0)
       (effects (font (size 1.27 1.27)) hide)
     )
@@
       (effects (font (size 1.27 1.27)))
     )
-    (property "Footprint" "Backplane:ZX SPECTRUM EDGE CONNECTOR (HORIZONTAL)" (at 68.58 157.48 0)
+    (property "Footprint" "Backplane_2:ZX SPECTRUM EDGE CONNECTOR (HORIZONTAL)" (at 68.58 157.48 0)
       (effects (font (size 1.27 1.27)) hide)
     )
@@
       (effects (font (size 1.27 1.27)) (justify left))
     )
-    (property "Footprint" "Connector_PinHeader_2.54mm:PinHeader_1x03_P2.54mm_Vertical" (at 242.57 140.97 0)
+    (property "Footprint" "Backplane_2:PinHeader_1x03_P2.54mm_Vertical" (at 242.57 140.97 0)
       (effects (font (size 1.27 1.27)) hide)
     )
@@
       (effects (font (size 1.27 1.27)))
     )
-    (property "Footprint" "Backplane:snp59_96_female_angle_3" (at 255.27 24.13 0)
+    (property "Footprint" "Backplane_2:snp59_96_female_angle_3" (at 255.27 24.13 0)
       (effects (font (size 1.27 1.27)) hide)
     )
@@
       (effects (font (size 1.27 1.27)))
     )
-    (property "Footprint" "Backplane:snp_straight" (at 41.91 24.13 0)
+    (property "Footprint" "Backplane_2:snp_straight" (at 41.91 24.13 0)
       (effects (font (size 1.27 1.27)) hide)
     )
@@
     )
   )
-  (symbol (lib_id "backplane_2:zx_bus") (at 129.54 157.48 0) (unit 1)
+  (symbol (lib_name "zx_bus_1") (lib_id "backplane_2:zx_bus") (at 129.54 157.48 0) (unit 1)
     (in_bom yes) (on_board yes) (dnp no) (fields_autoplaced)
     (property "Reference" "J7" (at 129.54 115.57 0)
@@
       (effects (font (size 1.27 1.27)))
     )
-    (property "Footprint" "Backplane:Spectrum_edge_slot_FIXED" (at 129.54 157.48 0)
+    (property "Footprint" "Backplane_2:Spectrum_edge_slot_FIXED" (at 129.54 157.48 0)
       (effects (font (size 1.27 1.27)) hide)
     )
@@
       (effects (font (size 1.27 1.27)))
     )
-    (property "Footprint" "Backplane:snp59_96_male_straight" (at 95.25 24.13 0)
+    (property "Footprint" "Backplane_2:snp59_96_male_straight" (at 95.25 24.13 0)
       (effects (font (size 1.27 1.27)) hide)
     )
@@
       (effects (font (size 1.27 1.27)) (justify left))
     )
-    (property "Footprint" "Capacitor_THT:CP_Radial_D8.0mm_P5.00mm" (at 210.5152 142.24 0)
+    (property "Footprint" "Backplane_2:CP_Radial_D8.0mm_P5.00mm" (at 210.5152 142.24 0)
       (effects (font (size 1.27 1.27)) hide)
     )
@@
       (effects (font (size 1.27 1.27)))
     )
-    (property "Footprint" "Backplane:snp59_96_male_straight" (at 147.32 24.13 0)
+    (property "Footprint" "Backplane_2:snp59_96_male_straight" (at 147.32 24.13 0)
       (effects (font (size 1.27 1.27)) hide)
     )
@@
       (effects (font (size 1.27 1.27)) (justify left))
     )
-    (property "Footprint" "Connector_PinHeader_2.54mm:PinHeader_1x04_P2.54mm_Vertical" (at 258.445 150.495 0)
+    (property "Footprint" "Backplane_2:PinHeader_1x04_P2.54mm_Vertical" (at 258.445 150.495 0)
       (effects (font (size 1.27 1.27)) hide)
     )
